Commit message: Add exact RealSense camera optical frames

File: ros2_ws/src/vla_lab_description/urdf/vla_lab_description.urdf (robot description, URDF)
Before this commit: robot vla_lab_description, 1 links, 0 joints
Links:
- added link d435i_link
- added link depth_camera_optical_frame
- added link left_ir_camera_optical_frame
- added link rgb_camera_optical_frame
- added link right_ir_camera_optical_frame
Joints:
- added joint d435i_joint: type fixed, parent vla_lab_base_link, child d435i_link, origin xyz=0.52326 0 0.75876 rpy=0 1.0143 -3.1416
- added joint depth_camera_optical_joint: type fixed, parent d435i_link, child depth_camera_optical_frame, origin xyz=0.012 0.0175 0 rpy=-1.5707963267949 0 -1.5707963267949
- added joint left_ir_camera_optical_joint: type fixed, parent d435i_link, child left_ir_camera_optical_frame, origin xyz=0.012 0.0175 0 rpy=-1.5707963267949 0 -1.5707963267949
- added joint rgb_camera_optical_joint: type fixed, parent d435i_link, child rgb_camera_optical_frame, origin xyz=0.012 0.0325 0 rpy=-1.5707963267949 0 -1.5707963267949
- added joint right_ir_camera_optical_joint: type fixed, parent d435i_link, child right_ir_camera_optical_frame, origin xyz=0.012 -0.0325 0 rpy=-1.5707963267949 0 -1.5707963267949
